File: DebugCAN.sch (EAGLE design)
At the start: 57 parts, among them J1 8P8C-LED, J2 XT60PW-M, J3 MA04-1, J4 10118192-0001LF, J5 8P8C-LED, J6 8P8C-LED, J7 8P8C-LED, U1 STM32F302C, U2 NCV7351D1E, U3 SI8621AB-B-IS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

Commit message: final update.
Parts:
- removed J2: XT60PW-M, con-xt:XT60PW-M
Connections:
- net +12V: no longer J2.2
- net GNDIO: no longer J2.GND
Changed lines of the file:
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@@
 <part name="J4" library="con-usb" deviceset="10118192-0001LF" device=""/>
 <part name="P+14" library="supply1" library_urn="urn:adsk.eagle:library:371" deviceset="+5V" device=""/>
-<part name="GND7" library="supply1" library_urn="urn:adsk.eagle:library:371" deviceset="GNDIO" device=""/>
-<part name="P+3" library="supply1" library_urn="urn:adsk.eagle:library:371" deviceset="+12V" device=""/>
-<part name="J2" library="con-xt" deviceset="XT60PW-M" device=""/>
 <part name="R10" library="rcl" library_urn="urn:adsk.eagle:library:334" deviceset="R-EU_" device="R0603" package3d_urn="urn:adsk.eagle:package:23555/3" value="470"/>
 <part name="R12" library="rcl" library_urn="urn:adsk.eagle:library:334" deviceset="R-EU_" device="R0603" package3d_urn="urn:adsk.eagle:package:23555/3" value="470"/>
@@
 <attribute name="VALUE" x="116.332" y="15.3162" size="1.778" layer="96"/>
 </instance>
-<instance part="GND7" gate="G$1" x="236.22" y="63.5" smashed="yes" rot="R270">
-<attribute name="VALUE" x="233.68" y="66.04" size="1.778" layer="96" rot="R270"/>
-</instance>
-<instance part="P+3" gate="1" x="236.22" y="58.42" smashed="yes" rot="R90">
-<attribute name="VALUE" x="241.3" y="55.88" size="1.778" layer="96" rot="R180"/>
-</instance>
-<instance part="J2" gate="G$1" x="254" y="60.96" smashed="yes">
-<attribute name="NAME" x="248.91255" y="66.68338125" size="1.780609375" layer="95"/>
-<attribute name="VALUE" x="248.9118" y="53.327709375" size="1.78086875" layer="96"/>
-</instance>
 <instance part="R10" gate="G$1" x="35.56" y="160.02" smashed="yes">
 <attribute name="NAME" x="31.75" y="161.5186" size="1.778" layer="95"/>
@@
 <pinref part="U6" gate="G$1" pin="C"/>
 </segment>
-<segment>
-<pinref part="J2" gate="G$1" pin="GND"/>
-<pinref part="GND7" gate="G$1" pin="GNDIO"/>
-<wire x1="243.84" y1="63.5" x2="238.76" y2="63.5" width="0.1524" layer="91"/>
-</segment>
 </net>
 <net name="N$3" class="0">
@@
 <pinref part="P+13" gate="1" pin="+12V"/>
 </segment>
-<segment>
-<pinref part="J2" gate="G$1" pin="2"/>
-<pinref part="P+3" gate="1" pin="+12V"/>
-<wire x1="243.84" y1="58.42" x2="238.76" y2="58.42" width="0.1524" layer="91"/>
-</segment>
 </net>
