File: DebugCAN.sch (EAGLE design)
At the start: 57 parts, among them J1 8P8C-LED, J3 MA04-1, J4 10118192-0001LF, J5 8P8C-LED, J6 8P8C-LED, J7 8P8C-LED, J8 XT60PW-F, U1 STM32F302C, U2 NCV7351D1E, U3 SI8621AB-B-IS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

Commit message: renew position
Parts:
- removed J8: XT60PW-F, con-xt:XT60PW-F
- added J2: XT60PW-M, con-xt:XT60PW-M
- C3, C4: value (none) -> 100n
- D1: value (none) -> GREEN
- D2: value (none) -> YELLOW
- D3: value (none) -> RED
- R1, R11, R13, R9: value (none) -> 1k
- R10, R12, R14, R2: value (none) -> 470
Connections:
- net +12V: now also J2.2; no longer J8.1
- net GNDIO: now also J2.GND; no longer J8.GND
Changed lines of the file:
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@@
 </variantdefs>
 <classes>
-<class number="0" name="default" width="0" drill="0">
+<class number="0" name="default" width="0.25" drill="0">
 </class>
 <class number="1" name="wide" width="0.5" drill="0">
+</class>
+<class number="2" name="6A" width="1.5" drill="0">
 </class>
 </classes>
@@
 <part name="GND5" library="supply1" library_urn="urn:adsk.eagle:library:371" deviceset="GNDIO" device=""/>
 <part name="GND6" library="supply1" library_urn="urn:adsk.eagle:library:371" deviceset="GNDIO" device=""/>
-<part name="R1" library="rcl" library_urn="urn:adsk.eagle:library:334" deviceset="R-EU_" device="R0603" package3d_urn="urn:adsk.eagle:package:23555/3"/>
-<part name="R2" library="rcl" library_urn="urn:adsk.eagle:library:334" deviceset="R-EU_" device="R0603" package3d_urn="urn:adsk.eagle:package:23555/3"/>
-<part name="C3" library="rcl" library_urn="urn:adsk.eagle:library:334" deviceset="C-EU" device="C0603" package3d_urn="urn:adsk.eagle:package:23616/2"/>
+<part name="R1" library="rcl" library_urn="urn:adsk.eagle:library:334" deviceset="R-EU_" device="R0603" package3d_urn="urn:adsk.eagle:package:23555/3" value="1k"/>
+<part name="R2" library="rcl" library_urn="urn:adsk.eagle:library:334" deviceset="R-EU_" device="R0603" package3d_urn="urn:adsk.eagle:package:23555/3" value="470"/>
+<part name="C3" library="rcl" library_urn="urn:adsk.eagle:library:334" deviceset="C-EU" device="C0603" package3d_urn="urn:adsk.eagle:package:23616/2" value="100n"/>
 <part name="GND8" library="supply1" library_urn="urn:adsk.eagle:library:371" deviceset="GNDIO" device=""/>
 <part name="H2" library="holes" library_urn="urn:adsk.eagle:library:237" deviceset="MOUNT-HOLE" device="3.2" package3d_urn="urn:adsk.eagle:package:14275/1"/>
@@
 <part name="C1" library="rcl" library_urn="urn:adsk.eagle:library:334" deviceset="CPOL-EU" device="153CLV-0605" package3d_urn="urn:adsk.eagle:package:23398/2" value="EEEHA1E220P"/>
 <part name="GND9" library="supply1" library_urn="urn:adsk.eagle:library:371" deviceset="GNDIO" device=""/>
-<part name="C4" library="rcl" library_urn="urn:adsk.eagle:library:334" deviceset="C-EU" device="C0603" package3d_urn="urn:adsk.eagle:package:23616/2"/>
+<part name="C4" library="rcl" library_urn="urn:adsk.eagle:library:334" deviceset="C-EU" device="C0603" package3d_urn="urn:adsk.eagle:package:23616/2" value="100n"/>
 <part name="GND22" library="supply1" library_urn="urn:adsk.eagle:library:371" deviceset="GNDIO" device=""/>
 <part name="+3V2" library="supply1" library_urn="urn:adsk.eagle:library:371" deviceset="+3V3" device=""/>
@@
 <part name="R6" library="rcl" deviceset="R-EU_" device="R0603" value="1k"/>
 <part name="R7" library="rcl" deviceset="R-EU_" device="R0603" value="1k"/>
-<part name="D1" library="led" library_urn="urn:adsk.eagle:library:259" deviceset="LED" device="CHIPLED_0805" package3d_urn="urn:adsk.eagle:package:15821/2"/>
-<part name="D2" library="led" library_urn="urn:adsk.eagle:library:259" deviceset="LED" device="CHIPLED_0805" package3d_urn="urn:adsk.eagle:package:15821/2"/>
-<part name="D3" library="led" library_urn="urn:adsk.eagle:library:259" deviceset="LED" device="CHIPLED_0805" package3d_urn="urn:adsk.eagle:package:15821/2"/>
+<part name="D1" library="led" library_urn="urn:adsk.eagle:library:259" deviceset="LED" device="CHIPLED_0805" package3d_urn="urn:adsk.eagle:package:15821/2" value="GREEN"/>
+<part name="D2" library="led" library_urn="urn:adsk.eagle:library:259" deviceset="LED" device="CHIPLED_0805" package3d_urn="urn:adsk.eagle:package:15821/2" value="YELLOW"/>
+<part name="D3" library="led" library_urn="urn:adsk.eagle:library:259" deviceset="LED" device="CHIPLED_0805" package3d_urn="urn:adsk.eagle:package:15821/2" value="RED"/>
 <part name="R8" library="rcl" deviceset="R-EU_" device="R0603" value="1k"/>
 <part name="GND28" library="supply1" library_urn="urn:adsk.eagle:library:371" deviceset="GNDA" device=""/>
@@
 <part name="GND36" library="supply1" library_urn="urn:adsk.eagle:library:371" deviceset="GNDIO" device=""/>
 <part name="GND37" library="supply1" library_urn="urn:adsk.eagle:library:371" deviceset="GNDIO" device=""/>
-<part name="R9" library="rcl" library_urn="urn:adsk.eagle:library:334" deviceset="R-EU_" device="R0603" package3d_urn="urn:adsk.eagle:package:23555/3"/>
-<part name="R10" library="rcl" library_urn="urn:adsk.eagle:library:334" deviceset="R-EU_" device="R0603" package3d_urn="urn:adsk.eagle:package:23555/3"/>
+<part name="R9" library="rcl" library_urn="urn:adsk.eagle:library:334" deviceset="R-EU_" device="R0603" package3d_urn="urn:adsk.eagle:package:23555/3" value="1k"/>
+<part name="R10" library="rcl" library_urn="urn:adsk.eagle:library:334" deviceset="R-EU_" device="R0603" package3d_urn="urn:adsk.eagle:package:23555/3" value="470"/>
 <part name="GND38" library="supply1" library_urn="urn:adsk.eagle:library:371" deviceset="GNDIO" device=""/>
 <part name="P+6" library="supply1" library_urn="urn:adsk.eagle:library:371" deviceset="+12V" device=""/>
@@
 <part name="GND42" library="supply1" library_urn="urn:adsk.eagle:library:371" deviceset="GNDIO" device=""/>
 <part name="GND43" library="supply1" library_urn="urn:adsk.eagle:library:371" deviceset="GNDIO" device=""/>
-<part name="R11" library="rcl" library_urn="urn:adsk.eagle:library:334" deviceset="R-EU_" device="R0603" package3d_urn="urn:adsk.eagle:package:23555/3"/>
-<part name="R12" library="rcl" library_urn="urn:adsk.eagle:library:334" deviceset="R-EU_" device="R0603" package3d_urn="urn:adsk.eagle:package:23555/3"/>
+<part name="R11" library="rcl" library_urn="urn:adsk.eagle:library:334" deviceset="R-EU_" device="R0603" package3d_urn="urn:adsk.eagle:package:23555/3" value="1k"/>
+<part name="R12" library="rcl" library_urn="urn:adsk.eagle:library:334" deviceset="R-EU_" device="R0603" package3d_urn="urn:adsk.eagle:package:23555/3" value="470"/>
 <part name="GND44" library="supply1" library_urn="urn:adsk.eagle:library:371" deviceset="GNDIO" device=""/>
 <part name="P+9" library="supply1" library_urn="urn:adsk.eagle:library:371" deviceset="+12V" device=""/>
@@
 <part name="GND48" library="supply1" library_urn="urn:adsk.eagle:library:371" deviceset="GNDIO" device=""/>
 <part name="GND49" library="supply1" library_urn="urn:adsk.eagle:library:371" deviceset="GNDIO" device=""/>
-<part name="R13" library="rcl" library_urn="urn:adsk.eagle:library:334" deviceset="R-EU_" device="R0603" package3d_urn="urn:adsk.eagle:package:23555/3"/>
-<part name="R14" library="rcl" library_urn="urn:adsk.eagle:library:334" deviceset="R-EU_" device="R0603" package3d_urn="urn:adsk.eagle:package:23555/3"/>
+<part name="R13" library="rcl" library_urn="urn:adsk.eagle:library:334" deviceset="R-EU_" device="R0603" package3d_urn="urn:adsk.eagle:package:23555/3" value="1k"/>
+<part name="R14" library="rcl" library_urn="urn:adsk.eagle:library:334" deviceset="R-EU_" device="R0603" package3d_urn="urn:adsk.eagle:package:23555/3" value="470"/>
 <part name="GND50" library="supply1" library_urn="urn:adsk.eagle:library:371" deviceset="GNDIO" device=""/>
 <part name="P+12" library="supply1" library_urn="urn:adsk.eagle:library:371" deviceset="+12V" device=""/>
@@
 <part name="J4" library="con-usb" deviceset="10118192-0001LF" device=""/>
 <part name="P+14" library="supply1" library_urn="urn:adsk.eagle:library:371" deviceset="+5V" device=""/>
-<part name="J8" library="con-xt" deviceset="XT60PW-F" device=""/>
 <part name="GND7" library="supply1" library_urn="urn:adsk.eagle:library:371" deviceset="GNDIO" device=""/>
+<part name="P+3" library="supply1" library_urn="urn:adsk.eagle:library:371" deviceset="+12V" device=""/>
+<part name="J2" library="con-xt" deviceset="XT60PW-M" device=""/>
 </parts>
 <sheets>
@@
 <attribute name="VALUE" x="116.332" y="15.3162" size="1.778" layer="96"/>
 </instance>
-<instance part="J8" gate="G$1" x="251.46" y="40.64" smashed="yes">
-<attribute name="NAME" x="246.37255" y="46.36338125" size="1.780609375" layer="95"/>
-<attribute name="VALUE" x="246.3718" y="33.007709375" size="1.78086875" layer="96"/>
-</instance>
-<instance part="GND7" gate="G$1" x="231.14" y="38.1" smashed="yes" rot="R270">
-<attribute name="VALUE" x="228.6" y="40.64" size="1.778" layer="96" rot="R270"/>
+<instance part="GND7" gate="G$1" x="236.22" y="63.5" smashed="yes" rot="R270">
+<attribute name="VALUE" x="233.68" y="66.04" size="1.778" layer="96" rot="R270"/>
+</instance>
+<instance part="P+3" gate="1" x="236.22" y="58.42" smashed="yes" rot="R90">
+<attribute name="VALUE" x="241.3" y="55.88" size="1.778" layer="96" rot="R180"/>
+</instance>
+<instance part="J2" gate="G$1" x="254" y="60.96" smashed="yes">
+<attribute name="NAME" x="248.91255" y="66.68338125" size="1.780609375" layer="95"/>
+<attribute name="VALUE" x="248.9118" y="53.327709375" size="1.78086875" layer="96"/>
 </instance>
 </instances>
@@
 </segment>
 <segment>
-<pinref part="J8" gate="G$1" pin="GND"/>
+<pinref part="J2" gate="G$1" pin="GND"/>
 <pinref part="GND7" gate="G$1" pin="GNDIO"/>
-<wire x1="241.3" y1="38.1" x2="233.68" y2="38.1" width="0.1524" layer="91"/>
+<wire x1="243.84" y1="63.5" x2="238.76" y2="63.5" width="0.1524" layer="91"/>
 </segment>
 </net>
@@
 </segment>
 </net>
-<net name="+12V" class="1">
+<net name="+12V" class="2">
 <segment>
 <pinref part="P+8" gate="1" pin="+12V"/>
@@
 </segment>
 <segment>
-<pinref part="J8" gate="G$1" pin="1"/>
-<wire x1="241.3" y1="43.18" x2="236.22" y2="43.18" width="0.1524" layer="91"/>
-<label x="236.22" y="43.18" size="1.778" layer="95" rot="R180" xref="yes"/>
+<pinref part="J2" gate="G$1" pin="2"/>
+<pinref part="P+3" gate="1" pin="+12V"/>
+<wire x1="243.84" y1="58.42" x2="238.76" y2="58.42" width="0.1524" layer="91"/>
 </segment>
 </net>

Commit message: led_regiser_changed
Parts:
- removed R10, R12, R14: 470, rcl:R-EU_R0603
Connections:
- removed net N$10: J5.C-Y, R10.2
- removed net N$13: J6.C-Y, R12.2
- removed net N$15: J7.C-Y, R14.2
- removed net N$4: J1.C-Y, R2.2
- new net CAN_LED_MPU: R2.1, U1.PB4-JNTRST
- net CAN_LED: now also R2.2; no longer U1.PB4-JNTRST
- net GNDA: now also J1.C-Y, J5.C-Y, J6.C-Y, J7.C-Y; no longer R10.1, R12.1, R14.1, R2.1
Other:
- moved on the sheet: R2
Changed lines of the file:
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@@
 <part name="GND37" library="supply1" library_urn="urn:adsk.eagle:library:371" deviceset="GNDIO" device=""/>
 <part name="R9" library="rcl" library_urn="urn:adsk.eagle:library:334" deviceset="R-EU_" device="R0603" package3d_urn="urn:adsk.eagle:package:23555/3" value="1k"/>
-<part name="R10" library="rcl" library_urn="urn:adsk.eagle:library:334" deviceset="R-EU_" device="R0603" package3d_urn="urn:adsk.eagle:package:23555/3" value="470"/>
 <part name="GND38" library="supply1" library_urn="urn:adsk.eagle:library:371" deviceset="GNDIO" device=""/>
 <part name="P+6" library="supply1" library_urn="urn:adsk.eagle:library:371" deviceset="+12V" device=""/>
@@
 <part name="GND43" library="supply1" library_urn="urn:adsk.eagle:library:371" deviceset="GNDIO" device=""/>
 <part name="R11" library="rcl" library_urn="urn:adsk.eagle:library:334" deviceset="R-EU_" device="R0603" package3d_urn="urn:adsk.eagle:package:23555/3" value="1k"/>
-<part name="R12" library="rcl" library_urn="urn:adsk.eagle:library:334" deviceset="R-EU_" device="R0603" package3d_urn="urn:adsk.eagle:package:23555/3" value="470"/>
 <part name="GND44" library="supply1" library_urn="urn:adsk.eagle:library:371" deviceset="GNDIO" device=""/>
 <part name="P+9" library="supply1" library_urn="urn:adsk.eagle:library:371" deviceset="+12V" device=""/>
@@
 <part name="GND49" library="supply1" library_urn="urn:adsk.eagle:library:371" deviceset="GNDIO" device=""/>
 <part name="R13" library="rcl" library_urn="urn:adsk.eagle:library:334" deviceset="R-EU_" device="R0603" package3d_urn="urn:adsk.eagle:package:23555/3" value="1k"/>
-<part name="R14" library="rcl" library_urn="urn:adsk.eagle:library:334" deviceset="R-EU_" device="R0603" package3d_urn="urn:adsk.eagle:package:23555/3" value="470"/>
 <part name="GND50" library="supply1" library_urn="urn:adsk.eagle:library:371" deviceset="GNDIO" device=""/>
 <part name="P+12" library="supply1" library_urn="urn:adsk.eagle:library:371" deviceset="+12V" device=""/>
@@
 <attribute name="VALUE" x="158.75" y="19.558" size="1.778" layer="96"/>
 </instance>
-<instance part="R2" gate="G$1" x="162.56" y="12.7" smashed="yes">
-<attribute name="NAME" x="158.75" y="14.1986" size="1.778" layer="95"/>
-<attribute name="VALUE" x="158.75" y="9.398" size="1.778" layer="96"/>
+<instance part="R2" gate="G$1" x="132.08" y="5.08" smashed="yes">
+<attribute name="NAME" x="128.27" y="6.5786" size="1.778" layer="95"/>
+<attribute name="VALUE" x="128.27" y="1.778" size="1.778" layer="96"/>
 </instance>
 <instance part="C3" gate="G$1" x="60.96" y="35.56" smashed="yes">
@@
 <attribute name="VALUE" x="34.29" y="166.878" size="1.778" layer="96"/>
 </instance>
-<instance part="R10" gate="G$1" x="38.1" y="160.02" smashed="yes">
-<attribute name="NAME" x="34.29" y="161.5186" size="1.778" layer="95"/>
-<attribute name="VALUE" x="34.29" y="156.718" size="1.778" layer="96"/>
-</instance>
 <instance part="GND38" gate="G$1" x="38.1" y="154.94" smashed="yes" rot="R270">
 <attribute name="VALUE" x="35.56" y="157.48" size="1.778" layer="96" rot="R270"/>
@@
 <attribute name="VALUE" x="148.59" y="169.418" size="1.778" layer="96"/>
 </instance>
-<instance part="R12" gate="G$1" x="152.4" y="162.56" smashed="yes">
-<attribute name="NAME" x="148.59" y="164.0586" size="1.778" layer="95"/>
-<attribute name="VALUE" x="148.59" y="159.258" size="1.778" layer="96"/>
-</instance>
 <instance part="GND44" gate="G$1" x="152.4" y="157.48" smashed="yes" rot="R270">
 <attribute name="VALUE" x="149.86" y="160.02" size="1.778" layer="96" rot="R270"/>
@@
 <attribute name="NAME" x="273.05" y="174.2186" size="1.778" layer="95"/>
 <attribute name="VALUE" x="273.05" y="169.418" size="1.778" layer="96"/>
-</instance>
-<instance part="R14" gate="G$1" x="276.86" y="162.56" smashed="yes">
-<attribute name="NAME" x="273.05" y="164.0586" size="1.778" layer="95"/>
-<attribute name="VALUE" x="273.05" y="159.258" size="1.778" layer="96"/>
 </instance>
 <instance part="GND50" gate="G$1" x="276.86" y="157.48" smashed="yes" rot="R270">
@@
 <pinref part="R1" gate="G$1" pin="2"/>
 <wire x1="167.64" y1="22.86" x2="170.18" y2="22.86" width="0.1524" layer="91"/>
-</segment>
-</net>
-<net name="N$4" class="0">
-<segment>
-<pinref part="J1" gate="G$1" pin="C-Y"/>
-<pinref part="R2" gate="G$1" pin="2"/>
-<wire x1="167.64" y1="12.7" x2="170.18" y2="12.7" width="0.1524" layer="91"/>
 </segment>
 </net>
@@
 </segment>
 </net>
-<net name="CAN_LED" class="0">
-<segment>
-<pinref part="J1" gate="G$1" pin="A-Y"/>
-<wire x1="170.18" y1="17.78" x2="139.7" y2="17.78" width="0.1524" layer="91"/>
-<wire x1="139.7" y1="17.78" x2="139.7" y2="5.08" width="0.1524" layer="91"/>
-<wire x1="139.7" y1="5.08" x2="109.22" y2="5.08" width="0.1524" layer="91"/>
-<label x="111.76" y="5.08" size="1.778" layer="95"/>
-</segment>
-<segment>
-<pinref part="J6" gate="G$1" pin="A-Y"/>
-<wire x1="160.02" y1="167.64" x2="129.54" y2="167.64" width="0.1524" layer="91"/>
-<label x="129.54" y="167.64" size="1.778" layer="95" rot="R180"/>
-</segment>
-<segment>
-<pinref part="J7" gate="G$1" pin="A-Y"/>
-<wire x1="284.48" y1="167.64" x2="254" y2="167.64" width="0.1524" layer="91"/>
-<label x="254" y="167.64" size="1.778" layer="95" rot="R180"/>
-</segment>
-<segment>
-<pinref part="J5" gate="G$1" pin="A-Y"/>
-<wire x1="45.72" y1="165.1" x2="15.24" y2="165.1" width="0.1524" layer="91"/>
-<label x="15.24" y="165.1" size="1.778" layer="95" rot="R180"/>
+<net name="CAN_LED_MPU" class="0">
+<segment>
+<pinref part="R2" gate="G$1" pin="1"/>
+<wire x1="127" y1="5.08" x2="116.84" y2="5.08" width="0.1524" layer="91"/>
+<label x="116.84" y="5.08" size="1.778" layer="95" rot="R180"/>
 </segment>
 </net>
@@
 </segment>
 <segment>
-<pinref part="R2" gate="G$1" pin="1"/>
-<wire x1="157.48" y1="12.7" x2="152.4" y2="12.7" width="0.1524" layer="91"/>
+<pinref part="GND39" gate="1" pin="GNDA"/>
+<pinref part="J5" gate="G$1" pin="C-Y"/>
+<wire x1="27.94" y1="160.02" x2="45.72" y2="160.02" width="0.1524" layer="91"/>
+</segment>
+<segment>
+<pinref part="GND45" gate="1" pin="GNDA"/>
+<pinref part="J6" gate="G$1" pin="C-Y"/>
+<wire x1="142.24" y1="162.56" x2="160.02" y2="162.56" width="0.1524" layer="91"/>
+</segment>
+<segment>
+<pinref part="GND51" gate="1" pin="GNDA"/>
+<pinref part="J7" gate="G$1" pin="C-Y"/>
+<wire x1="284.48" y1="162.56" x2="266.7" y2="162.56" width="0.1524" layer="91"/>
+</segment>
+<segment>
+<pinref part="J1" gate="G$1" pin="C-Y"/>
 <pinref part="GND31" gate="1" pin="GNDA"/>
-</segment>
-<segment>
-<pinref part="R10" gate="G$1" pin="1"/>
-<wire x1="33.02" y1="160.02" x2="27.94" y2="160.02" width="0.1524" layer="91"/>
-<pinref part="GND39" gate="1" pin="GNDA"/>
-</segment>
-<segment>
-<pinref part="R12" gate="G$1" pin="1"/>
-<wire x1="147.32" y1="162.56" x2="142.24" y2="162.56" width="0.1524" layer="91"/>
-<pinref part="GND45" gate="1" pin="GNDA"/>
-</segment>
-<segment>
-<pinref part="R14" gate="G$1" pin="1"/>
-<wire x1="271.78" y1="162.56" x2="266.7" y2="162.56" width="0.1524" layer="91"/>
-<pinref part="GND51" gate="1" pin="GNDA"/>
+<wire x1="170.18" y1="12.7" x2="152.4" y2="12.7" width="0.1524" layer="91"/>
 </segment>
 </net>
@@
 </segment>
 </net>
-<net name="N$10" class="0">
-<segment>
-<pinref part="J5" gate="G$1" pin="C-Y"/>
-<pinref part="R10" gate="G$1" pin="2"/>
-<wire x1="43.18" y1="160.02" x2="45.72" y2="160.02" width="0.1524" layer="91"/>
-</segment>
-</net>
 <net name="N$12" class="0">
 <segment>
@@
 </segment>
 </net>
-<net name="N$13" class="0">
-<segment>
-<pinref part="J6" gate="G$1" pin="C-Y"/>
-<pinref part="R12" gate="G$1" pin="2"/>
-<wire x1="157.48" y1="162.56" x2="160.02" y2="162.56" width="0.1524" layer="91"/>
-</segment>
-</net>
 <net name="N$14" class="0">
 <segment>
@@
 <pinref part="R13" gate="G$1" pin="2"/>
 <wire x1="281.94" y1="172.72" x2="284.48" y2="172.72" width="0.1524" layer="91"/>
-</segment>
-</net>
-<net name="N$15" class="0">
-<segment>
-<pinref part="J7" gate="G$1" pin="C-Y"/>
-<pinref part="R14" gate="G$1" pin="2"/>
-<wire x1="281.94" y1="162.56" x2="284.48" y2="162.56" width="0.1524" layer="91"/>
 </segment>
 </net>
@@
 <wire x1="60.96" y1="73.66" x2="96.52" y2="73.66" width="0.1524" layer="91"/>
 <label x="71.12" y="73.66" size="1.778" layer="95"/>
+</segment>
+</net>
+<net name="CAN_LED" class="0">
+<segment>
+<pinref part="J1" gate="G$1" pin="A-Y"/>
+<wire x1="170.18" y1="17.78" x2="139.7" y2="17.78" width="0.1524" layer="91"/>
+<wire x1="139.7" y1="17.78" x2="139.7" y2="5.08" width="0.1524" layer="91"/>
+<pinref part="R2" gate="G$1" pin="2"/>
+<wire x1="139.7" y1="5.08" x2="139.7" y2="0" width="0.1524" layer="91"/>
+<wire x1="139.7" y1="5.08" x2="137.16" y2="5.08" width="0.1524" layer="91"/>
+<junction x="139.7" y="5.08"/>
+<label x="139.7" y="0" size="1.778" layer="95"/>
+</segment>
+<segment>
+<pinref part="J5" gate="G$1" pin="A-Y"/>
+<wire x1="45.72" y1="165.1" x2="15.24" y2="165.1" width="0.1524" layer="91"/>
+<label x="15.24" y="165.1" size="1.778" layer="95" rot="R180"/>
+</segment>
+<segment>
+<pinref part="J6" gate="G$1" pin="A-Y"/>
+<wire x1="160.02" y1="167.64" x2="129.54" y2="167.64" width="0.1524" layer="91"/>
+<label x="129.54" y="167.64" size="1.778" layer="95" rot="R180"/>
+</segment>
+<segment>
+<pinref part="J7" gate="G$1" pin="A-Y"/>
+<wire x1="284.48" y1="167.64" x2="254" y2="167.64" width="0.1524" layer="91"/>
+<label x="254" y="167.64" size="1.778" layer="95" rot="R180"/>
 </segment>
 </net>
@@
 </segment>
 </net>
-<net name="CAN_LED" class="0">
+<net name="CAN_LED_MPU" class="0">
 <segment>
 <pinref part="U1" gate="G$1" pin="PB4-JNTRST"/>
