File: DebugCAN.sch (EAGLE design)
At the start: 54 parts, among them J1 8P8C-LED, J2 XT60PW-M, J3 MA04-1, J4 10118192-0001LF, J5 8P8C-LED, J6 8P8C-LED, J7 8P8C-LED, U1 STM32F302C, U2 NCV7351D1E, U3 SI8621AB-B-IS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

Commit message: fainal adjustment
Parts:
- added R10, R12, R14: 470, rcl:R-EU_R0603
- renumbered D2 to GNDA
Connections:
- removed net CAN_LED_MPU: R2.1, U1.PB4-JNTRST
- new net N$10: J5.C-Y, R10.2
- new net N$13: J6.C-Y, R12.2
- new net N$15: J7.C-Y, R14.2
- new net N$4: J1.C-Y, R2.2
- net CAN_LED: now also U1.PB4-JNTRST; no longer R2.2
- net GNDA: now also R10.1, R12.1, R14.1, R2.1; no longer J1.C-Y, J5.C-Y, J6.C-Y, J7.C-Y
Other:
- moved on the sheet: R2
Changed lines of the file:
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@@
 <part name="R7" library="rcl" deviceset="R-EU_" device="R0603" value="1k"/>
 <part name="D1" library="led" library_urn="urn:adsk.eagle:library:259" deviceset="LED" device="CHIPLED_0805" package3d_urn="urn:adsk.eagle:package:15821/2" value="GREEN"/>
-<part name="D2" library="led" library_urn="urn:adsk.eagle:library:259" deviceset="LED" device="CHIPLED_0805" package3d_urn="urn:adsk.eagle:package:15821/2" value="YELLOW"/>
+<part name="GNDA" library="led" library_urn="urn:adsk.eagle:library:259" deviceset="LED" device="CHIPLED_0805" package3d_urn="urn:adsk.eagle:package:15821/2" value="YELLOW"/>
 <part name="D3" library="led" library_urn="urn:adsk.eagle:library:259" deviceset="LED" device="CHIPLED_0805" package3d_urn="urn:adsk.eagle:package:15821/2" value="RED"/>
 <part name="R8" library="rcl" deviceset="R-EU_" device="R0603" value="1k"/>
@@
 <part name="P+3" library="supply1" library_urn="urn:adsk.eagle:library:371" deviceset="+12V" device=""/>
 <part name="J2" library="con-xt" deviceset="XT60PW-M" device=""/>
+<part name="R10" library="rcl" library_urn="urn:adsk.eagle:library:334" deviceset="R-EU_" device="R0603" package3d_urn="urn:adsk.eagle:package:23555/3" value="470"/>
+<part name="R12" library="rcl" library_urn="urn:adsk.eagle:library:334" deviceset="R-EU_" device="R0603" package3d_urn="urn:adsk.eagle:package:23555/3" value="470"/>
+<part name="R14" library="rcl" library_urn="urn:adsk.eagle:library:334" deviceset="R-EU_" device="R0603" package3d_urn="urn:adsk.eagle:package:23555/3" value="470"/>
 </parts>
 <sheets>
@@
 <attribute name="VALUE" x="158.75" y="19.558" size="1.778" layer="96"/>
 </instance>
-<instance part="R2" gate="G$1" x="132.08" y="5.08" smashed="yes">
-<attribute name="NAME" x="128.27" y="6.5786" size="1.778" layer="95"/>
-<attribute name="VALUE" x="128.27" y="1.778" size="1.778" layer="96"/>
+<instance part="R2" gate="G$1" x="162.56" y="12.7" smashed="yes">
+<attribute name="NAME" x="158.75" y="14.1986" size="1.778" layer="95"/>
+<attribute name="VALUE" x="158.75" y="9.398" size="1.778" layer="96"/>
 </instance>
 <instance part="C3" gate="G$1" x="60.96" y="35.56" smashed="yes">
@@
 <attribute name="NAME" x="248.91255" y="66.68338125" size="1.780609375" layer="95"/>
 <attribute name="VALUE" x="248.9118" y="53.327709375" size="1.78086875" layer="96"/>
+</instance>
+<instance part="R10" gate="G$1" x="35.56" y="160.02" smashed="yes">
+<attribute name="NAME" x="31.75" y="161.5186" size="1.778" layer="95"/>
+<attribute name="VALUE" x="31.75" y="156.718" size="1.778" layer="96"/>
+</instance>
+<instance part="R12" gate="G$1" x="149.86" y="162.56" smashed="yes">
+<attribute name="NAME" x="146.05" y="164.0586" size="1.778" layer="95"/>
+<attribute name="VALUE" x="146.05" y="159.258" size="1.778" layer="96"/>
+</instance>
+<instance part="R14" gate="G$1" x="274.32" y="162.56" smashed="yes">
+<attribute name="NAME" x="270.51" y="164.0586" size="1.778" layer="95"/>
+<attribute name="VALUE" x="270.51" y="159.258" size="1.778" layer="96"/>
 </instance>
 </instances>
@@
 </segment>
 </net>
-<net name="CAN_LED_MPU" class="0">
-<segment>
-<pinref part="R2" gate="G$1" pin="1"/>
-<wire x1="127" y1="5.08" x2="116.84" y2="5.08" width="0.1524" layer="91"/>
-<label x="116.84" y="5.08" size="1.778" layer="95" rot="R180"/>
-</segment>
-</net>
 <net name="+3V3" class="0">
 <segment>
@@
 </segment>
 <segment>
+<pinref part="R2" gate="G$1" pin="1"/>
+<pinref part="GND31" gate="1" pin="GNDA"/>
+<wire x1="157.48" y1="12.7" x2="152.4" y2="12.7" width="0.1524" layer="91"/>
+</segment>
+<segment>
+<pinref part="R10" gate="G$1" pin="1"/>
 <pinref part="GND39" gate="1" pin="GNDA"/>
-<pinref part="J5" gate="G$1" pin="C-Y"/>
-<wire x1="27.94" y1="160.02" x2="45.72" y2="160.02" width="0.1524" layer="91"/>
+<wire x1="30.48" y1="160.02" x2="27.94" y2="160.02" width="0.1524" layer="91"/>
 </segment>
 <segment>
 <pinref part="GND45" gate="1" pin="GNDA"/>
-<pinref part="J6" gate="G$1" pin="C-Y"/>
-<wire x1="142.24" y1="162.56" x2="160.02" y2="162.56" width="0.1524" layer="91"/>
-</segment>
-<segment>
+<pinref part="R12" gate="G$1" pin="1"/>
+<wire x1="142.24" y1="162.56" x2="144.78" y2="162.56" width="0.1524" layer="91"/>
+</segment>
+<segment>
+<pinref part="R14" gate="G$1" pin="1"/>
 <pinref part="GND51" gate="1" pin="GNDA"/>
-<pinref part="J7" gate="G$1" pin="C-Y"/>
-<wire x1="284.48" y1="162.56" x2="266.7" y2="162.56" width="0.1524" layer="91"/>
-</segment>
-<segment>
-<pinref part="J1" gate="G$1" pin="C-Y"/>
-<pinref part="GND31" gate="1" pin="GNDA"/>
-<wire x1="170.18" y1="12.7" x2="152.4" y2="12.7" width="0.1524" layer="91"/>
+<wire x1="269.24" y1="162.56" x2="266.7" y2="162.56" width="0.1524" layer="91"/>
 </segment>
 </net>
@@
 <wire x1="170.18" y1="17.78" x2="139.7" y2="17.78" width="0.1524" layer="91"/>
 <wire x1="139.7" y1="17.78" x2="139.7" y2="5.08" width="0.1524" layer="91"/>
-<pinref part="R2" gate="G$1" pin="2"/>
-<wire x1="139.7" y1="5.08" x2="139.7" y2="0" width="0.1524" layer="91"/>
-<wire x1="139.7" y1="5.08" x2="137.16" y2="5.08" width="0.1524" layer="91"/>
-<junction x="139.7" y="5.08"/>
-<label x="139.7" y="0" size="1.778" layer="95"/>
+<wire x1="139.7" y1="5.08" x2="119.38" y2="5.08" width="0.1524" layer="91"/>
+<label x="119.38" y="5.08" size="1.778" layer="95" rot="R180"/>
 </segment>
 <segment>
@@
 <wire x1="284.48" y1="167.64" x2="254" y2="167.64" width="0.1524" layer="91"/>
 <label x="254" y="167.64" size="1.778" layer="95" rot="R180"/>
+</segment>
+</net>
+<net name="N$4" class="0">
+<segment>
+<pinref part="J1" gate="G$1" pin="C-Y"/>
+<pinref part="R2" gate="G$1" pin="2"/>
+<wire x1="170.18" y1="12.7" x2="167.64" y2="12.7" width="0.1524" layer="91"/>
+</segment>
+</net>
+<net name="N$10" class="0">
+<segment>
+<pinref part="R10" gate="G$1" pin="2"/>
+<pinref part="J5" gate="G$1" pin="C-Y"/>
+<wire x1="40.64" y1="160.02" x2="45.72" y2="160.02" width="0.1524" layer="91"/>
+</segment>
+</net>
+<net name="N$13" class="0">
+<segment>
+<pinref part="R12" gate="G$1" pin="2"/>
+<pinref part="J6" gate="G$1" pin="C-Y"/>
+<wire x1="154.94" y1="162.56" x2="160.02" y2="162.56" width="0.1524" layer="91"/>
+</segment>
+</net>
+<net name="N$15" class="0">
+<segment>
+<pinref part="J7" gate="G$1" pin="C-Y"/>
+<pinref part="R14" gate="G$1" pin="2"/>
+<wire x1="284.48" y1="162.56" x2="279.4" y2="162.56" width="0.1524" layer="91"/>
 </segment>
 </net>
@@
 <attribute name="VALUE" x="253.492" y="92.075" size="1.778" layer="96" rot="R180"/>
 </instance>
-<instance part="D2" gate="G$1" x="248.92" y="78.74" smashed="yes" rot="R90">
+<instance part="GNDA" gate="G$1" x="248.92" y="78.74" smashed="yes" rot="R90">
 <attribute name="NAME" x="253.492" y="82.296" size="1.778" layer="95" rot="R180"/>
 <attribute name="VALUE" x="253.492" y="84.455" size="1.778" layer="96" rot="R180"/>
@@
 <segment>
 <pinref part="R7" gate="G$1" pin="2"/>
-<pinref part="D2" gate="G$1" pin="A"/>
+<pinref part="GNDA" gate="G$1" pin="A"/>
 <wire x1="243.84" y1="78.74" x2="246.38" y2="78.74" width="0.1524" layer="91"/>
 </segment>
@@
 <wire x1="256.54" y1="78.74" x2="256.54" y2="86.36" width="0.1524" layer="91"/>
 <wire x1="254" y1="86.36" x2="256.54" y2="86.36" width="0.1524" layer="91"/>
-<pinref part="D2" gate="G$1" pin="C"/>
+<pinref part="GNDA" gate="G$1" pin="C"/>
 <wire x1="254" y1="78.74" x2="256.54" y2="78.74" width="0.1524" layer="91"/>
 <junction x="256.54" y="78.74"/>
@@
 </segment>
 </net>
-<net name="CAN_LED_MPU" class="0">
+<net name="CAN_LED" class="0">
 <segment>
 <pinref part="U1" gate="G$1" pin="PB4-JNTRST"/>

Commit message: シルクの修正
Parts:
- renumbered GNDA to D2
Changed lines of the file:
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@@
 <part name="R7" library="rcl" deviceset="R-EU_" device="R0603" value="1k"/>
 <part name="D1" library="led" library_urn="urn:adsk.eagle:library:259" deviceset="LED" device="CHIPLED_0805" package3d_urn="urn:adsk.eagle:package:15821/2" value="GREEN"/>
-<part name="GNDA" library="led" library_urn="urn:adsk.eagle:library:259" deviceset="LED" device="CHIPLED_0805" package3d_urn="urn:adsk.eagle:package:15821/2" value="YELLOW"/>
+<part name="D2" library="led" library_urn="urn:adsk.eagle:library:259" deviceset="LED" device="CHIPLED_0805" package3d_urn="urn:adsk.eagle:package:15821/2" value="YELLOW"/>
 <part name="D3" library="led" library_urn="urn:adsk.eagle:library:259" deviceset="LED" device="CHIPLED_0805" package3d_urn="urn:adsk.eagle:package:15821/2" value="RED"/>
 <part name="R8" library="rcl" deviceset="R-EU_" device="R0603" value="1k"/>
@@
 <attribute name="VALUE" x="253.492" y="92.075" size="1.778" layer="96" rot="R180"/>
 </instance>
-<instance part="GNDA" gate="G$1" x="248.92" y="78.74" smashed="yes" rot="R90">
+<instance part="D2" gate="G$1" x="248.92" y="78.74" smashed="yes" rot="R90">
 <attribute name="NAME" x="253.492" y="82.296" size="1.778" layer="95" rot="R180"/>
 <attribute name="VALUE" x="253.492" y="84.455" size="1.778" layer="96" rot="R180"/>
@@
 <segment>
 <pinref part="R7" gate="G$1" pin="2"/>
-<pinref part="GNDA" gate="G$1" pin="A"/>
+<pinref part="D2" gate="G$1" pin="A"/>
 <wire x1="243.84" y1="78.74" x2="246.38" y2="78.74" width="0.1524" layer="91"/>
 </segment>
@@
 <wire x1="256.54" y1="78.74" x2="256.54" y2="86.36" width="0.1524" layer="91"/>
 <wire x1="254" y1="86.36" x2="256.54" y2="86.36" width="0.1524" layer="91"/>
-<pinref part="GNDA" gate="G$1" pin="C"/>
+<pinref part="D2" gate="G$1" pin="C"/>
 <wire x1="254" y1="78.74" x2="256.54" y2="78.74" width="0.1524" layer="91"/>
 <junction x="256.54" y="78.74"/>

Commit message: 突入電流対策
Parts:
- added F1: (no value), rcl:R-EU_R1206
Connections:
- new net N$1: F1.2, J2.2
- net +12V: now also F1.1; no longer J2.2
- net +5V_ISO: now also U$1.2; no longer U$1.1
- net EMS: now also U$1.1; no longer U$1.2
Changed lines of the file:
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@@
 <part name="R12" library="rcl" library_urn="urn:adsk.eagle:library:334" deviceset="R-EU_" device="R0603" package3d_urn="urn:adsk.eagle:package:23555/3" value="470"/>
 <part name="R14" library="rcl" library_urn="urn:adsk.eagle:library:334" deviceset="R-EU_" device="R0603" package3d_urn="urn:adsk.eagle:package:23555/3" value="470"/>
+<part name="F1" library="rcl" library_urn="urn:adsk.eagle:library:334" deviceset="R-EU_" device="R1206" package3d_urn="urn:adsk.eagle:package:23540/2"/>
 </parts>
 <sheets>
@@
 <attribute name="VALUE" x="233.68" y="66.04" size="1.778" layer="96" rot="R270"/>
 </instance>
-<instance part="P+3" gate="1" x="236.22" y="58.42" smashed="yes" rot="R90">
-<attribute name="VALUE" x="241.3" y="55.88" size="1.778" layer="96" rot="R180"/>
+<instance part="P+3" gate="1" x="226.06" y="58.42" smashed="yes" rot="R90">
+<attribute name="VALUE" x="231.14" y="55.88" size="1.778" layer="96" rot="R180"/>
 </instance>
 <instance part="J2" gate="G$1" x="254" y="60.96" smashed="yes">
@@
 <attribute name="NAME" x="270.51" y="164.0586" size="1.778" layer="95"/>
 <attribute name="VALUE" x="270.51" y="159.258" size="1.778" layer="96"/>
+</instance>
+<instance part="F1" gate="G$1" x="236.22" y="58.42" smashed="yes">
+<attribute name="NAME" x="232.41" y="59.9186" size="1.778" layer="95"/>
+<attribute name="VALUE" x="232.41" y="55.118" size="1.778" layer="96"/>
 </instance>
 </instances>
@@
 </segment>
 <segment>
-<pinref part="J2" gate="G$1" pin="2"/>
+<pinref part="F1" gate="G$1" pin="1"/>
 <pinref part="P+3" gate="1" pin="+12V"/>
-<wire x1="243.84" y1="58.42" x2="238.76" y2="58.42" width="0.1524" layer="91"/>
+<wire x1="231.14" y1="58.42" x2="228.6" y2="58.42" width="0.1524" layer="91"/>
 </segment>
 </net>
@@
 </segment>
 <segment>
-<wire x1="88.9" y1="48.26" x2="88.9" y2="38.1" width="0.1524" layer="91"/>
-<pinref part="U$1" gate="G$1" pin="1"/>
-<wire x1="88.9" y1="38.1" x2="86.36" y2="38.1" width="0.1524" layer="91"/>
-<label x="88.9" y="48.26" size="1.778" layer="95"/>
+<pinref part="U$1" gate="G$1" pin="2"/>
+<wire x1="86.36" y1="35.56" x2="93.98" y2="35.56" width="0.1524" layer="91"/>
+<label x="93.98" y="35.56" size="1.778" layer="95"/>
 </segment>
 </net>
@@
 </segment>
 <segment>
-<pinref part="U$1" gate="G$1" pin="2"/>
-<wire x1="86.36" y1="35.56" x2="91.44" y2="35.56" width="0.1524" layer="91"/>
-<label x="91.44" y="35.56" size="1.778" layer="95"/>
+<pinref part="U$1" gate="G$1" pin="1"/>
+<wire x1="86.36" y1="38.1" x2="91.44" y2="38.1" width="0.1524" layer="91"/>
+<label x="91.44" y="38.1" size="1.778" layer="95"/>
 </segment>
 </net>
@@
 </segment>
 </net>
+<net name="N$1" class="0">
+<segment>
+<pinref part="J2" gate="G$1" pin="2"/>
+<pinref part="F1" gate="G$1" pin="2"/>
+<wire x1="243.84" y1="58.42" x2="241.3" y2="58.42" width="0.1524" layer="91"/>
+</segment>
+</net>
