File: DebugCAN.brd (EAGLE design)
At the start: 56 x 63 mm, 57 parts, among them J1 8P8C-LED, J2 XT60PW-M, J3 MA04-1, J4 10118192-0001LF, J5 8P8C-LED, J6 8P8C-LED, J7 8P8C-LED, U1 STM32F302C, U2 NCV7351D1E, U3 SI8621AB-B-IS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

Commit message: led_regiser_changed
Parts:
- removed R10, R12, R14: 470, rcl:R0603
- moved R2 13.3 mm to (43.1, 37.1), flipped to the top, turned to 270 degrees
- moved TP2 0.75 mm to (40.7, 36.6)
- flipped C13 to the top, turned to 180 degrees
Connections:
- removed net N$10: J5.YC, R10.2
- removed net N$13: J6.YC, R12.2
- removed net N$15: J7.YC, R14.2
- removed net N$4: J1.YC, R2.2
- new net CAN_LED_MPU: R2.1, U1.40
- net CAN_LED: now also R2.2; no longer U1.40
- net GNDA: now also J1.YC, J5.YC, J6.YC, J7.YC; no longer R10.1, R12.1, R14.1, R2.1
Routing:
- net GNDA: track 0.00 -> 61.4 mm, vias 23 -> 56
- net N$4: track 35.0 -> 0.00 mm, vias 1 -> 0
- net N$15: track 30.1 -> 0.00 mm, vias 1 -> 0
- net N$13: track 15.9 -> 0.00 mm
- net CAN_LED: track 104.9 -> 93.0 mm
- net CAN_LED_MPU: track 0.00 -> 11.3 mm
- net N$10: track 7.68 -> 0.00 mm
- net +3V3: track 77.8 -> 77.2 mm

Commit message: fainal adjustment
Parts:
- removed D2: YELLOW, led:CHIPLED_0805
- added GNDA: YELLOW, led:CHIPLED_0805
- added R10, R12, R14: 470, rcl:R0603
- moved C8 3.25 mm to (41.9, 50.2), flipped to the top
- moved C14 1.91 mm to (25.0, 52.4), turned to 0 degrees
- moved R2 1.31 mm to (44.4, 36.8), turned to 180 degrees
- moved C10 0.97 mm to (43.3, 45.1), flipped to the top, turned to 180 degrees
- moved D1 0.25 mm to (53.7, 46.8)
- moved D3 0.25 mm to (53.7, 50.9)
- moved R6 0.25 mm to (48.0, 46.6)
- moved R7 0.25 mm to (48.0, 48.8)
- moved R8 0.25 mm to (48.0, 50.9)
Connections:
- removed net CAN_LED_MPU: R2.1, U1.40
- new net N$10: J5.YC, R10.2
- new net N$13: J6.YC, R12.2
- new net N$15: J7.YC, R14.2
- new net N$4: J1.YC, R2.2
- net CAN_LED: now also U1.40; no longer R2.2
- net GNDA: now also GNDA.C, R10.1, R12.1, R14.1, R2.1; no longer D2.C, J1.YC, J5.YC, J6.YC, J7.YC
- net N$2: now also GNDA.A; no longer D2.A
Routing:
- net GNDA: track 61.4 -> 0.24 mm, vias 56 -> 188
- net N$15: track 0.00 -> 33.5 mm, vias 0 -> 1
- net N$4: track 0.00 -> 26.7 mm
- net N$13: track 0.00 -> 13.5 mm
- net N$10: track 0.00 -> 11.5 mm
- net CAN_LED_MPU: track 11.3 -> 0.00 mm
- net CAN_LED: track 93.0 -> 102.5 mm
- net EMS: track 130.2 -> 138.3 mm
- net +3V3: track 77.2 -> 72.4 mm
- net CANH: track 107.2 -> 108.8 mm
- net CANL: track 106.9 -> 108.4 mm
- net +12V: track 107.9 -> 109.2 mm
- net +5V: track 10.1 -> 10.9 mm

Commit message: シルクの修正
Parts:
- renumbered GNDA to D2
Routing:
- net GNDA: vias 188 -> 193
Changed lines of the file:
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@@
 <drawing>
 <settings>
-<setting alwaysvectorfont="no"/>
+<setting alwaysvectorfont="yes"/>
 <setting verticaltext="up"/>
 </settings>
@@
 </element>
 <element name="C12" library="rcl" package="C0603" value="100n" x="41.605" y="39.34" smashed="yes" rot="MR270">
-<attribute name="NAME" x="38.65" y="34.845" size="1.27" layer="26" rot="MR180"/>
+<attribute name="NAME" x="40.65" y="42.845" size="1.27" layer="26" rot="MR180"/>
 <attribute name="VALUE" x="43.51" y="39.975" size="1.27" layer="28" rot="MR270"/>
 </element>
@@
 </element>
 <element name="C3" library="rcl" library_urn="urn:adsk.eagle:library:334" package="C0603" package3d_urn="urn:adsk.eagle:package:23616/2" value="100n" x="28.68" y="20.455" smashed="yes" rot="R90">
-<attribute name="NAME" x="27.545" y="19.57" size="1.27" layer="25" rot="R90"/>
+<attribute name="NAME" x="29.545" y="22.57" size="1.27" layer="25" rot="R90"/>
 <attribute name="SPICEPREFIX" value="C" x="103.61" y="89.035" size="1.778" layer="27" rot="R90" display="off"/>
 <attribute name="VALUE" x="30.585" y="19.82" size="1.27" layer="27" rot="R90"/>
@@
 </element>
 <element name="C7" library="rcl" package="C0805" value="4u7" x="40.4" y="36.73" smashed="yes" rot="MR0">
-<attribute name="NAME" x="42.545" y="41.625" size="1.27" layer="26" rot="MR0"/>
+<attribute name="NAME" x="41.545" y="34.625" size="1.27" layer="26" rot="MR0"/>
 <attribute name="VALUE" x="41.67" y="34.19" size="1.27" layer="28" rot="MR0"/>
 </element>
@@
 <attribute name="VALUE" x="52.43" y="44.215" size="1.27" layer="27"/>
 </element>
-<element name="GNDA" library="led" library_urn="urn:adsk.eagle:library:259" package="CHIPLED_0805" package3d_urn="urn:adsk.eagle:package:15821/2" value="YELLOW" x="53.7" y="48.835" smashed="yes" rot="R270">
+<element name="D2" library="led" library_urn="urn:adsk.eagle:library:259" package="CHIPLED_0805" package3d_urn="urn:adsk.eagle:package:15821/2" value="YELLOW" x="53.7" y="48.835" smashed="yes" rot="R270">
 <attribute name="NAME" x="49.805" y="48.105" size="1.27" layer="25"/>
 <attribute name="VALUE" x="52.43" y="46.295" size="1.27" layer="27"/>
@@
 </element>
 <element name="U2" library="on-semi" package="SO08" package3d_urn="urn:adsk.eagle:package:15356/1" value="NCV7351D1E" x="14.12" y="58.69" smashed="yes" rot="MR270">
-<attribute name="NAME" x="16.525" y="61.482" size="1.27" layer="26" rot="MR0"/>
+<attribute name="NAME" x="16.525" y="54.482" size="1.27" layer="26" rot="MR0"/>
 <attribute name="VALUE" x="16.025" y="54.753" size="1.27" layer="28" rot="MR0"/>
 </element>
 <element name="U3" library="silabs" package="SO08" package3d_urn="urn:adsk.eagle:package:15356/1" value="SI8621AB-B-IS" x="21.87" y="58.6" smashed="yes" rot="MR270">
-<attribute name="NAME" x="23.775" y="61.267" size="1.27" layer="26" rot="MR0"/>
+<attribute name="NAME" x="23.775" y="54.267" size="1.27" layer="26" rot="MR0"/>
 <attribute name="VALUE" x="23.775" y="54.663" size="1.27" layer="28" rot="MR0"/>
 </element>
@@
 </element>
 <element name="R12" library="rcl" library_urn="urn:adsk.eagle:library:334" package="R0603" package3d_urn="urn:adsk.eagle:package:23555/3" value="470" x="24.75" y="40.75" smashed="yes" rot="R270">
-<attribute name="NAME" x="22.385" y="42.385" size="1.27" layer="25" rot="R270"/>
+<attribute name="NAME" x="22.385" y="40.385" size="1.27" layer="25" rot="R270"/>
 <attribute name="POPULARITY" value="70" x="24.75" y="40.75" size="1.778" layer="27" rot="R270" display="off"/>
 <attribute name="SPICEPREFIX" value="R" x="24.75" y="40.75" size="1.778" layer="27" rot="R270" display="off"/>
@@
 </element>
 <element name="R14" library="rcl" library_urn="urn:adsk.eagle:library:334" package="R0603" package3d_urn="urn:adsk.eagle:package:23555/3" value="470" x="23.125" y="43.875" smashed="yes" rot="R270">
-<attribute name="NAME" x="23.76" y="44.51" size="1.27" layer="25" rot="R270"/>
+<attribute name="NAME" x="20.76" y="44.51" size="1.27" layer="25" rot="R270"/>
 <attribute name="POPULARITY" value="70" x="23.125" y="43.875" size="1.778" layer="27" rot="R270" display="off"/>
 <attribute name="SPICEPREFIX" value="R" x="23.125" y="43.875" size="1.778" layer="27" rot="R270" display="off"/>
@@
 <via x="18" y="50" extent="1-16" drill="0.35"/>
 <via x="2" y="43" extent="1-16" drill="0.35"/>
+<via x="39" y="15" extent="1-16" drill="0.35"/>
+<via x="32" y="11" extent="1-16" drill="0.35"/>
+<via x="25" y="11" extent="1-16" drill="0.35"/>
 </signal>
 <signal name="N$3">
@@
 <wire x1="35.21" y1="46.8278" x2="28.8602" y2="53.1776" width="0.25" layer="1"/>
 <wire x1="28.6102" y1="53.1776" x2="28.8602" y2="53.1776" width="0.25" layer="1"/>
-<wire x1="26.9608" y1="57.7444" x2="26.9608" y2="55.202" width="0.25" layer="16"/>
+<wire x1="27.2108" y1="57.4944" x2="27.2108" y2="54.952" width="0.25" layer="16"/>
 <wire x1="28.6102" y1="53.1776" x2="28.6102" y2="53.5526" width="0.25" layer="16"/>
-<wire x1="28.6102" y1="53.5526" x2="26.9608" y2="55.202" width="0.25" layer="16"/>
-<wire x1="25.5524" y1="59.1528" x2="26.9608" y2="57.7444" width="0.25" layer="16"/>
+<wire x1="28.6102" y1="53.5526" x2="27.2108" y2="54.952" width="0.25" layer="16"/>
+<wire x1="25.5524" y1="59.1528" x2="27.2108" y2="57.4944" width="0.25" layer="16"/>
 <wire x1="24.2446" y1="59.1528" x2="25.5524" y2="59.1528" width="0.25" layer="16"/>
 <wire x1="35.21" y1="45.8736" x2="35.19" y2="45.79" width="0.25" layer="1"/>
@@
 <contactref element="U1" pad="45"/>
 <wire x1="35.713" y1="47.0016" x2="35.713" y2="45.8736" width="0.25" layer="1"/>
-<wire x1="26.5584" y1="56.1562" x2="35.713" y2="47.0016" width="0.25" layer="1"/>
-<wire x1="26.5584" y1="57.2414" x2="26.5584" y2="56.1562" width="0.25" layer="1"/>
-<wire x1="26.3572" y1="57.4426" x2="26.5584" y2="57.2414" width="0.25" layer="1"/>
+<wire x1="27.1834" y1="55.5312" x2="35.713" y2="47.0016" width="0.25" layer="1"/>
+<wire x1="27.1834" y1="56.6164" x2="27.1834" y2="55.5312" width="0.25" layer="1"/>
+<wire x1="26.3572" y1="57.4426" x2="27.1834" y2="56.6164" width="0.25" layer="1"/>
 <wire x1="25.8542" y1="57.9456" x2="26.3572" y2="57.4426" width="0.25" layer="16"/>
 <wire x1="24.2446" y1="57.9456" x2="25.8542" y2="57.9456" width="0.25" layer="16"/>
@@
 <contactref element="U3" pad="4"/>
 <contactref element="D1" pad="C"/>
-<contactref element="GNDA" pad="C"/>
+<contactref element="D2" pad="C"/>
 <contactref element="D3" pad="C"/>
 <contactref element="U1" pad="23"/>
@@
 <via x="55.375" y="45.125" extent="1-16" drill="0.35"/>
 <via x="55.375" y="44.125" extent="1-16" drill="0.35"/>
+<via x="26.5" y="54.375" extent="1-16" drill="0.35"/>
+<via x="26.375" y="56.125" extent="1-16" drill="0.35"/>
+<via x="39" y="44" extent="1-16" drill="0.35"/>
+<via x="39" y="42" extent="1-16" drill="0.35"/>
+<via x="40" y="40" extent="1-16" drill="0.35"/>
 </signal>
 <signal name="N$9">
@@
 <signal name="N$2">
 <contactref element="R7" pad="2"/>
-<contactref element="GNDA" pad="A"/>
+<contactref element="D2" pad="A"/>
 <wire x1="52.562" y1="48.791" x2="48.8398" y2="48.791" width="0.25" layer="1"/>
 <wire x1="48.8398" y1="48.791" x2="48.815" y2="48.755" width="0.25" layer="1"/>

Commit message: 突入電流対策
Parts:
- added F1: (no value), rcl:R1206
- moved C1 5.75 mm to (27.5, 25.4)
- moved U5 3.00 mm to (21.2, 21.2)
- moved C3 1.98 mm to (29.6, 18.7), turned to 0 degrees
- moved U$1 1.50 mm to (51.5, 14.3), turned to 0 degrees
Connections:
- new net N$1: F1.2, J2.2
- net +12V: now also F1.1; no longer J2.2
- net +5V_ISO: now also U$1.P$2; no longer U$1.P$1
- net EMS: now also U$1.P$1; no longer U$1.P$2
Routing:
- net +12V: track 109.2 -> 105.2 mm
- net N$1: track 0.00 -> 3.85 mm
- net +5V_ISO: track 86.3 -> 89.3 mm
- net GNDA: vias 193 -> 194

Commit message: change F1
Parts:
- moved F1 7.00 mm to (26.9, 22.8)
- moved C1 5.62 mm to (33.2, 25.4)
- moved R16 1.41 mm to (24.5, 31.9), turned to 270 degrees
Connections:
- removed net N$1: F1.2, J2.2
- new net DCIN: C1.+, F1.2, J2.2
- net +12V: no longer C1.+
Routing:
- net DCIN: track 0.00 -> 10.9 mm
- net +12V: track 105.2 -> 98.2 mm
- net N$1: track 3.85 -> 0.00 mm
- net EMS: track 138.3 -> 135.6 mm
Changed lines of the file:
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@@
 <drawing>
 <settings>
-<setting alwaysvectorfont="yes"/>
+<setting alwaysvectorfont="no"/>
 <setting verticaltext="up"/>
 </settings>
@@
 </groups>
 <elements>
-<element name="C1" library="rcl" library_urn="urn:adsk.eagle:library:334" package="153CLV-0605" package3d_urn="urn:adsk.eagle:package:23398/2" value="EEEHA1E220P" x="27.54" y="25.425" smashed="yes" rot="R270">
-<attribute name="NAME" x="29.42" y="30.94" size="1.27" layer="25" rot="R270"/>
-<attribute name="SPICEPREFIX" value="C" x="-16.91" y="-8.865" size="1.778" layer="27" rot="R270" display="off"/>
-<attribute name="VALUE" x="22.655" y="28.85" size="1.27" layer="27" rot="R270"/>
+<element name="C1" library="rcl" library_urn="urn:adsk.eagle:library:334" package="153CLV-0605" package3d_urn="urn:adsk.eagle:package:23398/2" value="EEEHA1E220P" x="33.165" y="25.425" smashed="yes" rot="R270">
+<attribute name="NAME" x="35.045" y="30.94" size="1.27" layer="25" rot="R270"/>
+<attribute name="SPICEPREFIX" value="C" x="-11.285" y="-8.865" size="1.778" layer="27" rot="R270" display="off"/>
+<attribute name="VALUE" x="28.28" y="28.85" size="1.27" layer="27" rot="R270"/>
 </element>
 <element name="C10" library="rcl" package="C0603" value="100n" x="43.27" y="45.085" smashed="yes" rot="R180">
@@
 <attribute name="VALUE" x="25.295" y="19.705" size="1.27" layer="28" rot="MR180"/>
 </element>
-<element name="R16" library="rcl" library_urn="urn:adsk.eagle:library:334" package="R0603" package3d_urn="urn:adsk.eagle:package:23555/3" value="470" x="23.63" y="30.79" smashed="yes">
-<attribute name="NAME" x="21.995" y="32.3" size="1.27" layer="25"/>
-<attribute name="POPULARITY" value="70" x="52.84" y="-40.33" size="1.778" layer="27" display="off"/>
-<attribute name="SPICEPREFIX" value="R" x="52.84" y="-40.33" size="1.778" layer="27" display="off"/>
-<attribute name="VALUE" x="22.995" y="28.885" size="1.27" layer="27"/>
+<element name="R16" library="rcl" library_urn="urn:adsk.eagle:library:334" package="R0603" package3d_urn="urn:adsk.eagle:package:23555/3" value="470" x="24.54" y="31.87" smashed="yes" rot="R270">
+<attribute name="NAME" x="26.05" y="33.505" size="1.27" layer="25" rot="R270"/>
+<attribute name="POPULARITY" value="70" x="-46.58" y="2.66" size="1.778" layer="27" rot="R270" display="off"/>
+<attribute name="SPICEPREFIX" value="R" x="-46.58" y="2.66" size="1.778" layer="27" rot="R270" display="off"/>
+<attribute name="VALUE" x="22.635" y="32.505" size="1.27" layer="27" rot="R270"/>
 </element>
 <element name="R2" library="rcl" library_urn="urn:adsk.eagle:library:334" package="R0603" package3d_urn="urn:adsk.eagle:package:23555/3" value="470" x="44.365" y="36.76" smashed="yes" rot="R180">
@@
 <attribute name="VALUE" x="21.22" y="44.51" size="1.27" layer="27" rot="R270"/>
 </element>
-<element name="F1" library="rcl" library_urn="urn:adsk.eagle:library:334" package="R1206" package3d_urn="urn:adsk.eagle:package:23540/2" value="" x="33.875" y="22.75" smashed="yes">
-<attribute name="NAME" x="32.605" y="24.02" size="1.27" layer="25"/>
-<attribute name="POPULARITY" value="41" x="33.875" y="22.75" size="1.778" layer="27" display="off"/>
-<attribute name="SPICEPREFIX" value="R" x="33.875" y="22.75" size="1.778" layer="27" display="off"/>
-<attribute name="VALUE" x="32.605" y="20.21" size="1.27" layer="27"/>
+<element name="F1" library="rcl" library_urn="urn:adsk.eagle:library:334" package="R1206" package3d_urn="urn:adsk.eagle:package:23540/2" value="" x="26.875" y="22.75" smashed="yes">
+<attribute name="NAME" x="25.605" y="24.02" size="1.27" layer="25"/>
+<attribute name="POPULARITY" value="41" x="26.875" y="22.75" size="1.778" layer="27" display="off"/>
+<attribute name="SPICEPREFIX" value="R" x="26.875" y="22.75" size="1.778" layer="27" display="off"/>
+<attribute name="VALUE" x="25.605" y="20.21" size="1.27" layer="27"/>
 </element>
 </elements>
@@
 <via x="18" y="39" extent="1-16" drill="0.3048"/>
 <via x="34" y="29" extent="1-16" drill="0.35"/>
-<via x="28" y="28" extent="1-16" drill="0.35"/>
-<via x="28" y="27" extent="1-16" drill="0.35"/>
+<via x="33" y="29" extent="1-16" drill="0.35"/>
+<via x="33" y="27" extent="1-16" drill="0.35"/>
 <via x="36" y="29" extent="1-16" drill="0.35"/>
 <via x="30" y="29" extent="1-16" drill="0.35"/>
@@
 <contactref element="J1" pad="5"/>
 <contactref element="J1" pad="GA"/>
-<contactref element="C1" pad="+"/>
-<contactref element="U5" pad="3"/>
 <contactref element="J5" pad="4"/>
 <contactref element="J5" pad="5"/>
@@
 <wire x1="22.3512" y1="22.7356" x2="23.156" y2="22.7356" width="1.5" layer="1"/>
 <wire x1="22.3512" y1="22.7356" x2="21.8482" y2="23.2386" width="1.5" layer="1"/>
-<wire x1="23.156" y1="22.7356" x2="23.156" y2="22.694" width="1.5" layer="1"/>
 <wire x1="2.771" y1="39.9656" x2="7.419434375" y2="44.614034375" width="1.5" layer="1"/>
 <wire x1="2.771" y1="30.7104" x2="2.771" y2="39.9656" width="1.5" layer="1"/>
@@
 <wire x1="11.21039375" y1="24.8914" x2="14.76679375" y2="21.335" width="1.5" layer="1"/>
 <contactref element="F1" pad="1"/>
-<wire x1="23.156" y1="22.694" x2="27.509" y2="22.694" width="1.5" layer="1"/>
-<wire x1="27.509" y1="22.694" x2="27.54" y2="22.725" width="1.5" layer="1"/>
-<wire x1="32.453" y1="22.75" x2="27.565" y2="22.75" width="1.5" layer="1"/>
-<wire x1="27.565" y1="22.75" x2="27.54" y2="22.725" width="1.5" layer="1"/>
+<contactref element="U5" pad="3"/>
+<wire x1="23.156" y1="22.694" x2="25.397" y2="22.694" width="1.5" layer="1"/>
+<wire x1="25.397" y1="22.694" x2="25.453" y2="22.75" width="1.5" layer="1"/>
+<wire x1="23.156" y1="22.7356" x2="23.156" y2="22.694" width="0" layer="19" extent="1-1"/>
 </signal>
 <signal name="+5V_ISO" class="1">
@@
 <contactref element="J6" pad="6"/>
 <contactref element="J7" pad="6"/>
-<wire x1="25.778" y1="33.826" x2="25.778" y2="45.7547" width="0.25" layer="1"/>
-<wire x1="22.8362" y1="30.8842" x2="25.778" y2="33.826" width="0.25" layer="1"/>
-<wire x1="22.8362" y1="30.8842" x2="22.78" y2="30.79" width="0.25" layer="1"/>
 <wire x1="17.985" y1="10.595" x2="17.405" y2="10.595" width="0.25" layer="16"/>
 <wire x1="17.405" y1="10.595" x2="16.2812" y2="11.7188" width="0.25" layer="16"/>
@@
 <wire x1="33.25" y1="3.5" x2="34.6086" y2="4.8586" width="0.25" layer="1"/>
 <wire x1="34.6086" y1="4.8586" x2="34.6086" y2="9.2965125" width="0.25" layer="1"/>
-<wire x1="24.1561" y1="47.3766" x2="25.778" y2="45.7547" width="0.25" layer="1"/>
+<wire x1="25.778" y1="45.7547" x2="25.76635" y2="45.76635" width="0.25" layer="1"/>
 <contactref element="U$1" pad="P$1"/>
+<wire x1="25.76635" y1="45.76635" x2="24.1561" y2="47.3766" width="0.25" layer="1"/>
 <wire x1="52.71" y1="13.605" x2="52.705" y2="13.605" width="0.25" layer="16"/>
 <wire x1="52.705" y1="13.605" x2="51.1" y2="12" width="0.25" layer="16"/>
 <wire x1="37.94" y1="12" x2="51.1" y2="12" width="0.25" layer="16"/>
+<wire x1="25.76635" y1="45.76635" x2="25.76635" y2="33.94635" width="0.25" layer="1"/>
+<wire x1="25.76635" y1="33.94635" x2="24.54" y2="32.72" width="0.25" layer="1"/>
 </signal>
 <signal name="N$25">
@@
 <wire x1="24.5464" y1="30.8842" x2="24.647" y2="30.9848" width="0.25" layer="1"/>
 <wire x1="26.4578" y1="30.9848" x2="26.485" y2="31.025" width="0.25" layer="1"/>
-<wire x1="24.5464" y1="30.8842" x2="24.48" y2="30.79" width="0.25" layer="1"/>
+<wire x1="24.5464" y1="30.8842" x2="24.54" y2="31.02" width="0.25" layer="1"/>
 </signal>
 <signal name="!EMS">
@@
 <via x="13" y="46" extent="1-16" drill="0.35"/>
 </signal>
-<signal name="N$1">
+<signal name="DCIN" class="2">
+<contactref element="C1" pad="+"/>
+<wire x1="33.134" y1="22.694" x2="33.165" y2="22.725" width="1.5" layer="1"/>
+<wire x1="33.19" y1="22.75" x2="33.165" y2="22.725" width="1.5" layer="1"/>
+<contactref element="F1" pad="2"/>
 <contactref element="J2" pad="2"/>
-<contactref element="F1" pad="2"/>
-<wire x1="35.297" y1="22.75" x2="38.65" y2="22.75" width="1.7" layer="1"/>
-<wire x1="38.65" y1="22.75" x2="39" y2="22.4" width="1.7" layer="1"/>
+<wire x1="28.297" y1="22.75" x2="33.19" y2="22.75" width="1.5" layer="1"/>
+<wire x1="33.165" y1="22.725" x2="38.675" y2="22.725" width="1.5" layer="1"/>
+<wire x1="38.675" y1="22.725" x2="39" y2="22.4" width="1.5" layer="1"/>
 </signal>
 </signals>

Commit message: update
Routing:
- net +5V_ISO: track 89.3 -> 88.7 mm
Changed lines of the file:
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@@
 <wire x1="10.4624" y1="25.3512" x2="10.545" y2="25.325" width="1.5" layer="1"/>
 <wire x1="8.8528" y1="26.2566" x2="8.765" y2="26.345" width="1.5" layer="1"/>
-<wire x1="22.3512" y1="22.7356" x2="23.156" y2="22.7356" width="1.5" layer="1"/>
-<wire x1="22.3512" y1="22.7356" x2="21.8482" y2="23.2386" width="1.5" layer="1"/>
 <wire x1="2.771" y1="39.9656" x2="7.419434375" y2="44.614034375" width="1.5" layer="1"/>
 <wire x1="2.771" y1="30.7104" x2="2.771" y2="39.9656" width="1.5" layer="1"/>
@@
 <wire x1="24.015" y1="15.405" x2="24.015" y2="13.015" width="1.5" layer="1"/>
 <wire x1="24.015" y1="13.015" x2="24" y2="13" width="1.5" layer="1"/>
-<wire x1="17.41678125" y1="23.2386" x2="15.51318125" y2="21.335" width="1.5" layer="1"/>
-<wire x1="21.8482" y1="23.2386" x2="17.41678125" y2="23.2386" width="1.5" layer="1"/>
+<wire x1="15.51318125" y1="21.335" x2="17.41678125" y2="23.2386" width="1.5" layer="1"/>
 <wire x1="10.545" y1="25.325" x2="10.9786" y2="24.8914" width="1.5" layer="1"/>
 <wire x1="10.9786" y1="24.8914" x2="11.21039375" y2="24.8914" width="1.5" layer="1"/>
@@
 <wire x1="23.156" y1="22.694" x2="25.397" y2="22.694" width="1.5" layer="1"/>
 <wire x1="25.397" y1="22.694" x2="25.453" y2="22.75" width="1.5" layer="1"/>
-<wire x1="23.156" y1="22.7356" x2="23.156" y2="22.694" width="0" layer="19" extent="1-1"/>
+<wire x1="17.41678125" y1="23.2386" x2="21.9864" y2="23.2386" width="1.5" layer="1"/>
+<wire x1="22.531" y1="22.694" x2="23.156" y2="22.694" width="1.5" layer="1"/>
+<wire x1="22.531" y1="22.694" x2="21.9864" y2="23.2386" width="1.5" layer="1"/>
 </signal>
 <signal name="+5V_ISO" class="1">
@@
 <wire x1="19.5164" y1="60.5612" x2="19.52" y2="60.505" width="0.5" layer="16"/>
 <wire x1="15.6936" y1="58.1468" x2="16.47" y2="58.055" width="0.5" layer="16"/>
-<wire x1="23.156" y1="18.695" x2="28.73" y2="18.695" width="0.5" layer="1"/>
-<wire x1="23.156" y1="18.695" x2="23.156" y2="19.696" width="0.5" layer="1"/>
+<wire x1="24.156" y1="18.695" x2="28.73" y2="18.695" width="0.5" layer="1"/>
+<wire x1="24.156" y1="18.696" x2="23.156" y2="19.696" width="0.5" layer="1"/>
+<wire x1="24.156" y1="18.696" x2="24.156" y2="18.695" width="0.5" layer="1"/>
 <wire x1="28.9728" y1="18.9128" x2="29.4758" y2="18.9128" width="0.5" layer="16"/>
 <wire x1="28.5704" y1="18.5104" x2="28.9728" y2="18.9128" width="0.5" layer="16"/>
@@
 <wire x1="33.25" y1="3.5" x2="34.6086" y2="4.8586" width="0.25" layer="1"/>
 <wire x1="34.6086" y1="4.8586" x2="34.6086" y2="9.2965125" width="0.25" layer="1"/>
-<wire x1="25.778" y1="45.7547" x2="25.76635" y2="45.76635" width="0.25" layer="1"/>
 <contactref element="U$1" pad="P$1"/>
 <wire x1="25.76635" y1="45.76635" x2="24.1561" y2="47.3766" width="0.25" layer="1"/>
@@
 <signal name="DCIN" class="2">
 <contactref element="C1" pad="+"/>
-<wire x1="33.134" y1="22.694" x2="33.165" y2="22.725" width="1.5" layer="1"/>
-<wire x1="33.19" y1="22.75" x2="33.165" y2="22.725" width="1.5" layer="1"/>
 <contactref element="F1" pad="2"/>
 <contactref element="J2" pad="2"/>
-<wire x1="28.297" y1="22.75" x2="33.19" y2="22.75" width="1.5" layer="1"/>
+<wire x1="33.19" y1="22.75" x2="28.297" y2="22.75" width="1.5" layer="1"/>
 <wire x1="33.165" y1="22.725" x2="38.675" y2="22.725" width="1.5" layer="1"/>
 <wire x1="38.675" y1="22.725" x2="39" y2="22.4" width="1.5" layer="1"/>
+<wire x1="33.165" y1="22.725" x2="33.19" y2="22.75" width="1.5" layer="1"/>
 </signal>
 </signals>

Commit message: ver.2 update
Parts:
- moved F1 8.12 mm to (34.9, 21.4), turned to 270 degrees
- moved C1 3.09 mm to (30.2, 26.2)
- moved C3 1.35 mm to (29.6, 20.0)
- moved U5 1.00 mm to (22.2, 21.2)
Connections:
- net +12V: now also C1.+; no longer J1.4, J1.5, J1.GA, J5.4, J5.5, J5.GA, J6.4, J6.5, J6.GA, J7.4, J7.5, J7.GA
- net DCIN: now also J1.4, J1.5, J1.GA, J5.4, J5.5, J5.GA, J6.4, J6.5, J6.GA, J7.4, J7.5, J7.GA; no longer C1.+
Routing:
- net DCIN: track 10.9 -> 107.2 mm
- net +12V: track 98.2 -> 11.7 mm
- net +5V_ISO: track 88.7 -> 92.4 mm
